Commit message: 更新move_base 参数

File: rm_simulation/livox_laser_simulation/urdf/livox_mid360.xacro (robot description, xacro)
@@ -59,6 +59,6 @@
   </xacro:macro>
   <xacro:macro name="mid360" params="visualize:=True name:='livox' parent:='base_link' *origin">
-    <joint name="lidar_joint" type="fixed">
-        <axis xyz="0 1 0" />
+    <joint name="lidar_joint" type="continuous">
+        <axis xyz="0 0 1" />
         <xacro:insert_block name="origin"/>
         <parent link="${parent}"/>
